Commit message: update

File: robots/mp_500/mp_500.urdf (robot description, URDF)
Before this commit: robot mp_500, 6 links, 5 joints
Links:
- link base_link: geometry collision mesh filename=package://final_assessment/robots/mp_500/meshes/MP-500-BODY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 scale=0.001 0.001 0.001; visual mesh filename=package://final_assessment/robots/mp_500/meshes/MP-500-BODY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 scale=0.001 0.001 0.001
- link caster_wheel_link: geometry collision mesh filename=package://final_assessment/robots/mp_500/meshes/MP-500-WHEE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 scale=0.001 0.001 0.001; visual mesh filename=package://final_assessment/robots/mp_500/meshes/MP-500-WHEE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 scale=0.001 0.001 0.001
- link lidar_1_link: geometry collision mesh filename=package://final_assessment/components/sensors/SICK-S300.dae scale=0.001 0.001 0.001; visual mesh filename=package://final_assessment/components/sensors/SICK-S300.dae scale=0.001 0.001 0.001
- link wheel_left_link: geometry collision mesh filename=package://final_assessment/robots/mp_500/meshes/MP-500-WHEE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 scale=0.001 0.001 0.001; visual mesh filename=package://final_assessment/robots/mp_500/meshes/MP-500-WHEE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 scale=0.001 0.001 0.001
- link wheel_right_link: geometry collision mesh filename=package://final_assessment/robots/mp_500/meshes/MP-500-WHEE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 scale=0.001 0.001 0.001; visual mesh filename=package://final_assessment/robots/mp_500/meshes/MP-500-WHEE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 scale=0.001 0.001 0.001
